File: pcb/motdrive.kicad_sch (KiCad schematic)
At the start: 4 parts, among them J2 Conn_01x02, U3 DRV8837C

Commit message: complete overhaul wip
Parts:
- removed C1: 0.1uF, Capacitor_SMD:C_0402_1005Metric, symbol Device:C
- removed J2: Conn_01x02, Connector_PinHeader_1.27mm:PinHeader_1x02_P1.27mm_Vertical, symbol Connector_Generic:Conn_01x02
- removed U3: DRV8837C, Package_SON:WSON-8-1EP_2x2mm_P0.5mm_EP0.9x1.6mm, symbol Driver_Motor:DRV8837C
- added C16: 10uF, Capacitor_SMD:C_0402_1005Metric, symbol Device:C
- added C18: 0.1uF, Capacitor_SMD:C_0402_1005Metric, symbol Device:C
- added C20: 22nF, Capacitor_SMD:C_0402_1005Metric, symbol Device:C
- added R14, R15: 1, Resistor_SMD:R_0402_1005Metric, symbol Device:R
- added R20: 47k, Resistor_SMD:R_0402_1005Metric, symbol Device:R
- added R22: 1k, Resistor_SMD:R_0402_1005Metric, symbol Device:R
- added U5: STSPIN220, Package_DFN_QFN:VQFN-16-1EP_3x3mm_P0.5mm_EP1.8x1.8mm, symbol Driver_Motor:STSPIN220
- renumbered C3 to C17
Connections:
- net +3V3: now also U5.15 (MODE2)
- net GND: now also C16.2, C18.2, C20.2, R14.2, R15.2, R20.2, U5.16 (MODE1), U5.17 (EPAD), U5.7 (GND)
- net VDC: now also C16.1, U5.6 (VS); no longer C17.1
- new net: C20.1, R22.2
- new net: R15.1, U5.4 (SENSEA)
- new net: R14.1, U5.9 (SENSEB)
- new net: R20.1, R22.1, U5.12 (TOFF)
- new net DIR: U5.1 (DIR)
- new net EN: C17.1, U5.13 (EN/FLT)
- new net MOTA1: U5.3 (OUTA1)
- new net MOTA2: U5.5 (OUTA2)
- new net MOTB1: U5.10 (OUTB1)
- new net MOTB2: U5.8 (OUTB2)
- new net RST: C18.1, U5.14 (STBY/RESET)
- new net STEP: U5.2 (STCK)
- new net VREF: U5.11 (REF)
Other:
- moved on the sheet: C17

Commit message: lots of pcb work, test code, and final fw framework starting
Parts:
- removed R20: 47k, Resistor_SMD:R_0402_1005Metric, symbol Device:R
- added R24: 47k, Resistor_SMD:R_0402_1005Metric, symbol Device:R
- renumbered C18 to C16, C20 to C18, C17 to C19, C16 to C21, R22 to R16, R14 to R22, R15 to R23
Connections:
- net GND: now also R24.2
- net at R16.1, U5.12 (TOFF): now also R24.1

Commit message: getting close to order state
Connections:
- net GND: no longer U5.16 (MODE1)
- net +3V3 renamed MODE2
- new net MODE1: U5.16 (MODE1)
Changed lines of the file:
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@@
+    (stroke (width 0) (type default))
+  )
+  (wire (pts (xy 120.65 90.17) (xy 118.11 90.17))
     (stroke (width 0) (type default))
   )
@@
     (stroke (width 0) (type default))
   )
-  (wire (pts (xy 102.87 90.17) (xy 120.65 90.17))
-    (stroke (width 0) (type default))
-  )
   (wire (pts (xy 118.11 129.54) (xy 114.3 129.54))
     (stroke (width 0) (type default))
@@
     (stroke (width 0) (type default))
   )
+  (wire (pts (xy 120.65 92.71) (xy 118.11 92.71))
+    (stroke (width 0) (type default))
+  )
   (wire (pts (xy 118.11 115.57) (xy 118.11 111.76))
     (stroke (width 0) (type default))
@@
     (stroke (width 0) (type default))
   )
-  (wire (pts (xy 102.87 90.17) (xy 102.87 91.44))
-    (stroke (width 0) (type default))
-  )
   (wire (pts (xy 133.35 114.3) (xy 134.62 114.3))
     (stroke (width 0) (type default))
@@
     (stroke (width 0) (type default))
   )
-  (wire (pts (xy 120.65 92.71) (xy 106.68 92.71))
-    (stroke (width 0) (type default))
-  )
-  (wire (pts (xy 106.68 92.71) (xy 106.68 87.63))
-    (stroke (width 0) (type default))
-  )
   (wire (pts (xy 83.82 100.33) (xy 86.36 100.33))
     (stroke (width 0) (type default))
@@
   (wire (pts (xy 148.59 82.55) (xy 151.13 82.55))
     (stroke (width 0) (type default))
+  )
+  (hierarchical_label "MODE1" (shape input) (at 118.11 90.17 180) (fields_autoplaced)
+    (effects (font (size 1.27 1.27)) (justify right))
   )
   (hierarchical_label "VREF" (shape input) (at 118.11 105.41 180) (fields_autoplaced)
@@
     (effects (font (size 1.27 1.27)) (justify left))
   )
+  (hierarchical_label "MODE2" (shape input) (at 118.11 92.71 180) (fields_autoplaced)
+    (effects (font (size 1.27 1.27)) (justify right))
+  )
   (hierarchical_label "DIR" (shape input) (at 118.11 82.55 180) (fields_autoplaced)
     (effects (font (size 1.27 1.27)) (justify right))
@@
     )
   )
-  (symbol (lib_id "power:+3V3") (at 106.68 87.63 0) (unit 1)
-    (in_bom yes) (on_board yes) (dnp no) (fields_autoplaced)
-    (property "Reference" "#PWR057" (at 106.68 91.44 0)
-      (effects (font (size 1.27 1.27)) hide)
-    )
-    (property "Value" "+3V3" (at 106.68 82.55 0)
-      (effects (font (size 1.27 1.27)))
-    )
-    (property "Footprint" "" (at 106.68 87.63 0)
-      (effects (font (size 1.27 1.27)) hide)
-    )
-    (property "Datasheet" "" (at 106.68 87.63 0)
-      (effects (font (size 1.27 1.27)) hide)
-    )
-    (pin "1")
-    (instances
-      (project "MiniBot"
-        (path "/0e598331-3211-4e8a-a305-31a83585854d/30439bae-73bd-4041-a14b-0bcf2e025602"
-          (reference "#PWR057") (unit 1)
-        )
-        (path "/0e598331-3211-4e8a-a305-31a83585854d/5bde5315-a331-4fb7-9bbc-33e1b550bab8"
-          (reference "#PWR068") (unit 1)
-        )
-      )
-    )
-  )
   (symbol (lib_id "power:VDC") (at 88.9 72.39 0) (unit 1)
     (in_bom yes) (on_board yes) (dnp no) (fields_autoplaced)
@@
         )
       )
-    )
-  )
-  (symbol (lib_id "power:GND") (at 102.87 91.44 0) (unit 1)
-    (in_bom yes) (on_board yes) (dnp no) (fields_autoplaced)
-    (property "Reference" "#PWR056" (at 102.87 97.79 0)
-      (effects (font (size 1.27 1.27)) hide)
-    )
-    (property "Value" "GND" (at 102.87 96.52 0)
-      (effects (font (size 1.27 1.27)))
-    )
-    (property "Footprint" "" (at 102.87 91.44 0)
-      (effects (font (size 1.27 1.27)) hide)
-    )
-    (property "Datasheet" "" (at 102.87 91.44 0)
-      (effects (font (size 1.27 1.27)) hide)
-    )
-    (pin "1")
-    (instances
-      (project "MiniBot"
-        (path "/0e598331-3211-4e8a-a305-31a83585854d/30439bae-73bd-4041-a14b-0bcf2e025602"
-          (reference "#PWR056") (unit 1)
-        )
-        (path "/0e598331-3211-4e8a-a305-31a83585854d/5bde5315-a331-4fb7-9bbc-33e1b550bab8"
-          (reference "#PWR067") (unit 1)
-        )
-      )
