File: pcb/MiniBot.kicad_pcb (KiCad board)
At the start: 2 copper layers, 22.7 x 38.2 mm, 51 parts, among them IC1 MIC23050-SYML-TR, IC2 RT9527GQW, IC3 LM324QT, J1 GSB1C41110SSHR, J2 Conn_01x02, J3 Conn_01x02, J4 Conn_01x02, J5 Conn_01x02, J6 Conn_01x01, J7 Conn_01x01, U1 ESP32-C3-MINI-1-H4X, U3 DRV8837C, U4 DRV8837C

Commit message: big updates
Parts:
- removed D4: LED_Dual_KAKA, SamacSys_Parts:SB0603WC01-RG
- removed IC2: RT9527GQW, SamacSys_Parts:SON50P200X200X80-9N
- removed J6, J7: Conn_01x01, TestPoint:TestPoint_Pad_D1.0mm
- removed R16: 300, Resistor_SMD:R_0402_1005Metric
- added C14: 0.1uF, Capacitor_SMD:C_0402_1005Metric, F.Cu at (154.6, 63.6)
- added C15: 0.1uF, Capacitor_SMD:C_0402_1005Metric, F.Cu at (162.4, 46.2)
- added C16: 4.7uF, Capacitor_SMD:C_0402_1005Metric, F.Cu at (160.3, 67.6)
- added C17: 0.1uF, Capacitor_SMD:C_0402_1005Metric, F.Cu at (152.2, 65.6)
- added C18: 0.1uF, Capacitor_SMD:C_0402_1005Metric, F.Cu at (160.3, 68.6)
- added C19: 4.7uF, Capacitor_SMD:C_0402_1005Metric, F.Cu at (137.8, 52.9)
- added C20: 0.1uF, Capacitor_SMD:C_0402_1005Metric, F.Cu at (137.8, 54.9)
- added D2: LED, Diode_SMD:D_0402_1005Metric, F.Cu at (153.6, 65.0)
- added D3: LED, Diode_SMD:D_0402_1005Metric, F.Cu at (161.4, 41.4)
- added R21: 10k, Resistor_SMD:R_0402_1005Metric, F.Cu at (148.1, 57.1)
- added R22: 10k, Resistor_SMD:R_0402_1005Metric, F.Cu at (153.1, 46.9)
- added R25: 10k, Resistor_SMD:R_0402_1005Metric, F.Cu at (153.0, 67.9)
- added S3: SSU-121BRT, SamacSys_Parts:SSU121BRT, F.Cu at (146.5, 43.8)
- added U2: MCP73832-2-OT, Package_TO_SOT_SMD:SOT-23-5, F.Cu at (155.6, 67.4)
- C11: value 500nF -> 4.7uF
- C12: value 0.1uF -> 1uF
- C6, C7: value uF -> 0.001uF
- J2, J3: moved to B.Cu
- R14: value 4k -> 261
- R15: value 300 -> 1k
- moved R14 25.7 mm to (161.4, 42.4), turned to 0 degrees
- moved S1 19.8 mm to (145.8, 54.1)
- moved R18 15.7 mm to (163.4, 46.2)
- moved R17 14.8 mm to (161.4, 46.2), turned to -90 degrees
- moved C2 12.7 mm to (148.7, 68.3), turned to 0 degrees
- moved R4 12.3 mm to (159.3, 45.5), turned to 0 degrees
- moved C13 11.4 mm to (144.6, 58.4), turned to 180 degrees
- moved R20 11.4 mm to (146.4, 58.4), turned to 180 degrees
- moved C4 9.03 mm to (151.9, 63.6)
- moved C9 8.08 mm to (148.1, 59.0), turned to 90 degrees
- moved U4 7.63 mm to (149.8, 64.0), turned to 180 degrees
- moved S2 6.95 mm to (145.8, 50.1), turned to 180 degrees
- moved R3 6.88 mm to (155.0, 46.9), turned to 0 degrees
- moved R9 5.93 mm to (157.8, 46.1), turned to -90 degrees
- moved C7 5.49 mm to (156.9, 46.1), turned to -90 degrees
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Connections:
- C11 pad 1: Net-(IC2-TIMER) -> GND
- C11 pad 2: GND -> +BATT
- C8 pad 1: VDC -> +BATT
- J5 pad 2: VDC -> +BATT
- R14 pad 1: Net-(IC2-ISET) -> +3V3
- R14 pad 2: GND -> Net-(D3-A)
- R15 pad 1: +5V -> Net-(D2-K)
- U1 pad 12: unconnected-(U1-IO0-Pad12) -> /AMP
- U1 pad 16: /IO1 -> /M1_IN2
- U1 pad 18: /M_SLEEP -> /M1_IN1
- U1 pad 19: /M1_IN1 -> /M0_IN2
- U1 pad 20: /M1_IN2 -> /M0_IN1
- U1 pad 21: /M0_IN1 -> /M_SLEEP
- U1 pad 22: /M0_IN2 -> /GPIO8
- U1 pad 5: /AMP -> /GPIO2
- U1 pad 6: /IO0 -> unconnected-(U1-IO3-Pad6)
Routing:
- net GND: track 178.1 -> 91.8 mm
- net +BATT: track 0.00 -> 39.2 mm, vias 0 -> 2
- net VDC: track 58.9 -> 74.9 mm
- net /VSENSE: track 4.04 -> 15.8 mm, vias 0 -> 2
- net +3V3: track 73.1 -> 84.3 mm, vias 5 -> 8
- net /M1_IN2: track 3.28 -> 12.2 mm, vias 0 -> 2
- net Net-(J3-Pin_1): track 3.43 -> 11.2 mm, vias 0 -> 1
- net /M1_IN1: track 3.92 -> 11.1 mm, vias 0 -> 2
- net Net-(IC2-ISET): track 6.19 -> 0.00 mm
- net /GPIO2: track 0.00 -> 5.04 mm
- net Net-(J3-Pin_2): track 5.13 -> 10.2 mm, vias 0 -> 1
- net Net-(D4-A2): track 4.82 -> 0.00 mm
- net /Ultrasonic Amplifier/IN2+: track 10.8 -> 6.25 mm
- net /M0_IN2: track 7.71 -> 12.0 mm, vias 0 -> 2
- net /Ultrasonic Amplifier/IN2-: track 8.36 -> 4.17 mm
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- added copper zone on In2.Cu, net VDC
Other:
- board size 22.7 x 38.2 mm -> 22.7 x 37.2 mm
- copper layers 2 -> 4
- board text added: "3v3"
- board text added: "miniBOT"

Commit message: complete overhaul wip
Parts:
- removed D3: LED, Diode_SMD:D_0402_1005Metric
- removed IC3: LM324QT, SamacSys_Parts:QFN50P300X300X100-17N
- removed J4: Conn_01x02, SamacSys_Parts:Transducer
- removed J5: Conn_01x02, Connector_JST:JST_PH_S2B-PH-K_1x02_P2.00mm_Horizontal
- removed R17, R18: 390k, Resistor_SMD:R_0402_1005Metric
- removed R19: 10k, Resistor_SMD:R_0402_1005Metric
- added C21: 22nF, Capacitor_SMD:C_0402_1005Metric, F.Cu at (147.8, 75.0)
- added C22: 0.1uF, Capacitor_SMD:C_0402_1005Metric, F.Cu at (161.7, 62.6)
- added R23: 1k, Resistor_SMD:R_0402_1005Metric, F.Cu at (147.8, 74.0)
- added R24: 390k, Resistor_SMD:R_0402_1005Metric, F.Cu at (158.8, 62.7)
- added U5: STSPIN220, Package_DFN_QFN:VQFN-16-1EP_3x3mm_P0.5mm_EP1.8x1.8mm, F.Cu at (150.7, 71.3)
- C1: value 0.1uF -> 4.7uF
- C10: value 560pF -> 4.7uF
- C11, D2, IC1, U1: moved to B.Cu
- C12: value 1uF -> 0.1uF
- C14: value 0.1uF -> 10uF
- C16: value 4.7uF -> 10uF
- C19, C8: value 4.7uF -> 0.1uF
- C20: value 0.1uF -> 22nF
- C3: value 0.1uF -> 1uF
- C6: value 0.001uF -> 560pF
- C7: value 0.001uF -> 4.7uF
- D1: value D -> LED
- J1: value GSB1C41110SSHR -> Conn_01x08; footprint SamacSys_Parts:GSB1C41110SSHR -> Connector_JST:JST_SH_BM08B-SRSS-TB_1x08-1MP_P1.00mm_Vertical
- J2: footprint Connector_PinHeader_1.27mm:PinHeader_1x02_P1.27mm_Vertical -> Connector_JST:JST_PH_B2B-PH-K_1x02_P2.00mm_Vertical; moved to F.Cu
- J3: value Conn_01x02 -> GSB1C41110SSHR; footprint Connector_PinHeader_1.27mm:PinHeader_1x02_P1.27mm_Vertical -> SamacSys_Parts:GSB1C41110SSHR
- R1: value 4.7M -> 10k
- R10: value 1M -> 5.1k
- R11: value 4.7M -> 5.1k
- R12, R13: value 5.1k -> 1
- R14: value 261 -> 1
- R15: value 1k -> 1
- R2: value 1M -> 261
- R20, R21: value 10k -> 47k
- R22: value 10k -> 1k
- R25: value 10k -> 15k
- R3, R4: value 1M -> 10k
- R5: value 12K -> 10k
- R6: value 1M -> 390k
- R7: value 4.7M -> 390k
- R8: value 390k -> 10k; moved to B.Cu
- R9: value 12K -> 1k; moved to B.Cu
- S1: value EVP-AWBD4A -> SSU-121BRT; footprint SamacSys_Parts:EVPAWBD4A -> SamacSys_Parts:SSU121BRT
- S3: value SSU-121BRT -> EVP-AWBD4A; footprint SamacSys_Parts:SSU121BRT -> SamacSys_Parts:EVPAWBD4A
- U2: value MCP73832-2-OT -> TLV493D; footprint Package_TO_SOT_SMD:SOT-23-5 -> Package_TO_SOT_SMD:SOT-23-6
- U3: value DRV8837C -> MCP73832-2-OT; footprint Package_SON:WSON-8-1EP_2x2mm_P0.5mm_EP0.9x1.6mm -> Package_TO_SOT_SMD:SOT-23-5
- U4: value DRV8837C -> STSPIN220; footprint Package_SON:WSON-8-1EP_2x2mm_P0.5mm_EP0.9x1.6mm -> Package_DFN_QFN:VQFN-16-1EP_3x3mm_P0.5mm_EP1.8x1.8mm
- moved C8 68.1 mm to (92.9, 46.9), turned to 0 degrees
- moved C12 65.1 mm to (98.0, 53.6), turned to 0 degrees
- moved L1 63.0 mm to (94.9, 52.4)
- moved C15 61.6 mm to (100.8, 49.7), turned to 0 degrees
- moved C10 61.3 mm to (98.0, 49.7), turned to 0 degrees
- moved R4 57.8 mm to (104.0, 62.1)
- moved C14 56.1 mm to (100.8, 47.7), turned to 0 degrees
- moved R13 55.0 mm to (98.0, 57.6), turned to 0 degrees
- moved R12 54.1 mm to (98.0, 55.6), turned to 0 degrees
- moved R1 52.9 mm to (104.0, 56.2), turned to 0 degrees
- moved R3 52.7 mm to (104.0, 60.1)
- moved R6 52.3 mm to (104.0, 66.1), turned to 0 degrees
- moved D1 51.0 mm to (110.0, 62.1), turned to 0 degrees
- moved R5 50.2 mm to (104.0, 64.1), turned to 0 degrees
- moved R2 49.1 mm to (104.0, 58.1), turned to 0 degrees
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Connections:
- C1 pad 1: +3V3 -> GND
- C1 pad 2: GND -> +3V3
- C10 pad 1: +3V3 -> GND
- C10 pad 2: /CFF -> +BATT
- C11 pad 1: GND -> +3V3
- C11 pad 2: +BATT -> GND
- C12 pad 1: /RST -> +BATT
- C13 pad 1: /GPIO9 -> +3V3
- C14 pad 1: +3V3 -> VDC
- C15 pad 1: /VSENSE -> /MotorDriver1/EN
- C17 pad 1: +5V -> /MotorDriver0/EN
- C18 pad 1: +BATT -> /MotorDriver1/RST
- C19 pad 1: GND -> /MotorDriver0/RST
- C19 pad 2: +3V3 -> GND
- C20 pad 1: +3V3 -> Net-(C20-Pad1)
- C3 pad 1: VDC -> /RST
- C4 pad 1: VDC -> /GPIO9
- C5 pad 1: /Ultrasonic Amplifier/IN3- -> /VSENSE
- C6 pad 1: Net-(C6-Pad1) -> +3V3
- C6 pad 2: GND -> /CFF
- C7 pad 1: Net-(C7-Pad1) -> VDC
- C8 pad 1: +BATT -> +5V
- C9 pad 1: +3V3 -> +BATT
- D1 pad 1: /Ultrasonic Amplifier/OUT2 -> GND
- D2 pad 2: +5V -> +BATT
- J2 pad 1: Net-(J2-Pin_1) -> GND
- J2 pad 2: Net-(J2-Pin_2) -> +BATT
- R1 pad 1: Net-(D1-A) -> +3V3
- R1 pad 2: /Ultrasonic Amplifier/IN3- -> /RST
- R10 pad 1: /Ultrasonic Amplifier/OUT2 -> /CC1
- R10 pad 2: /Ultrasonic Amplifier/IN2- -> GND
- R11 pad 1: /AMP -> /CC2
- R11 pad 2: /Ultrasonic Amplifier/IN3+ -> GND
- R12 pad 1: /CC1 -> Net-(U4-SENSEB)
- R13 pad 1: /CC2 -> Net-(U4-SENSEA)
- R14 pad 1: +3V3 -> Net-(U5-SENSEB)
- R14 pad 2: Net-(D3-A) -> GND
- R15 pad 1: Net-(D2-K) -> Net-(U5-SENSEA)
- R15 pad 2: Net-(U2-STAT) -> GND
- R2 pad 1: /Ultrasonic Amplifier/IN2+ -> +3V3
- R2 pad 2: /Ultrasonic Amplifier/IN1- -> Net-(D1-A)
- R20 pad 1: +3V3 -> Net-(U4-TOFF)
- R20 pad 2: /GPIO9 -> GND
- R21 pad 1: +3V3 -> Net-(U5-TOFF)
- R21 pad 2: /GPIO8 -> GND
- R22 pad 1: +3V3 -> Net-(U4-TOFF)
- R22 pad 2: /GPIO2 -> Net-(C20-Pad1)
- R25 pad 1: Net-(U2-PROG) -> /VREF
- R3 pad 2: /Ultrasonic Amplifier/IN1+ -> /GPIO8
- R4 pad 1: /Ultrasonic Amplifier/IN1+ -> +3V3
- R4 pad 2: GND -> /GPIO2
- R5 pad 1: /Ultrasonic Amplifier/IN1- -> +3V3
- R5 pad 2: Net-(C6-Pad1) -> /GPIO9
- R6 pad 1: /Ultrasonic Amplifier/IN3+ -> VDC
- R6 pad 2: GND -> /VSENSE
- R7 pad 1: +3V3 -> /VSENSE
- R7 pad 2: /Ultrasonic Amplifier/IN3- -> GND
- R8 pad 1: +3V3 -> Net-(U3-PROG)
- R8 pad 2: /Ultrasonic Amplifier/IN3+ -> GND
- R9 pad 1: /Ultrasonic Amplifier/IN2- -> Net-(D2-K)
- R9 pad 2: Net-(C7-Pad1) -> Net-(U3-STAT)
- S1 pad A1: /RST -> unconnected-(S1-NC-PadA1)
- S1 pad A2: GND -> +5V
- S2 pad A1: /GPIO9 -> /RST
- S3 pad A1: unconnected-(S3-NC-PadA1) -> /GPIO9
- S3 pad A2: unconnected-(S3-PadA2) -> GND
- U1 pad 12: /AMP -> unconnected-(U1-IO0-Pad12)
- U1 pad 16: /M1_IN2 -> unconnected-(U1-IO10-Pad16)
- U1 pad 18: /M1_IN1 -> unconnected-(U1-IO4-Pad18)
- U1 pad 19: /M0_IN2 -> unconnected-(U1-IO5-Pad19)
- U1 pad 20: /M0_IN1 -> unconnected-(U1-IO6-Pad20)
- U1 pad 21: /M_SLEEP -> unconnected-(U1-IO7-Pad21)
- U1 pad 30: unconnected-(U1-RXD0-Pad30) -> /SDA
- U1 pad 31: unconnected-(U1-TXD0-Pad31) -> /SCL
- U2 pad 1: Net-(U2-STAT) -> /SCL
- U2 pad 3: +BATT -> GND
- U2 pad 4: +5V -> +3V3
- U2 pad 5: Net-(U2-PROG) -> GND
- U3 pad 1: VDC -> Net-(U3-STAT)
- U3 pad 2: Net-(J2-Pin_1) -> GND
- U3 pad 3: Net-(J2-Pin_2) -> +BATT
- U3 pad 4: GND -> +5V
- U3 pad 5: /M0_IN2 -> Net-(U3-PROG)
- U4 pad 1: VDC -> /MotorDriver1/DIR
- U4 pad 2: Net-(J3-Pin_1) -> /MotorDriver1/STEP
- U4 pad 3: Net-(J3-Pin_2) -> /M1_A1
- U4 pad 4: GND -> Net-(U4-SENSEA)
- U4 pad 5: /M1_IN2 -> /M1_A2
- U4 pad 6: /M1_IN1 -> VDC
- U4 pad 7: /M_SLEEP -> GND
- U4 pad 8: +3V3 -> /M1_B2
- U4 pad 9: GND -> Net-(U4-SENSEB)
Routing:
- net +3V3: track 84.3 -> 2.24 mm, vias 8 -> 0
- net VDC: track 74.9 -> 0.11 mm, vias 6 -> 0
- net GND: track 91.8 -> 18.1 mm, vias 37 -> 9
- net +BATT: track 39.2 -> 10.7 mm, vias 2 -> 1
- net /RST: track 24.5 -> 0.00 mm, vias 3 -> 0
- net /GPIO9: track 23.9 -> 0.00 mm, vias 3 -> 0
- net +5V: track 21.7 -> 1.44 mm, vias 4 -> 1
- net /M_SLEEP: track 17.3 -> 0.00 mm, vias 3 -> 0
- net /Ultrasonic Amplifier/IN1+: track 17.3 -> 0.00 mm, vias 5 -> 0
- net /VSENSE: track 15.8 -> 0.00 mm, vias 2 -> 0
- net /AMP: track 13.3 -> 0.00 mm, vias 2 -> 0
- net /M1_IN2: track 12.2 -> 0.00 mm, vias 2 -> 0
- net /M0_IN1: track 12.2 -> 0.00 mm, vias 2 -> 0
- net /M0_IN2: track 12.0 -> 0.00 mm, vias 2 -> 0
- net Net-(J3-Pin_1): track 11.2 -> 0.00 mm, vias 1 -> 0
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- removed copper zone on B.Cu, net GND
- removed copper zone on F.Cu, net GND
- removed copper zone on In2.Cu, net VDC
Other:
- board size 22.7 x 37.2 mm -> 27.9 x 28 mm
- board text removed: "3v3"
- board text removed: "BOOT"
- board text removed: "L R"
- board text removed: "RST"
- board text removed: "miniBOT"

Commit message: lots of pcb work, test code, and final fw framework starting
Parts:
- removed C11: 4.7uF, Capacitor_SMD:C_0402_1005Metric
- removed C12, C13: 0.1uF, Capacitor_SMD:C_0402_1005Metric
- removed C14: 10uF, Capacitor_SMD:C_0402_1005Metric
- removed R21: 47k, Resistor_SMD:R_0402_1005Metric
- removed U2: TLV493D, Package_TO_SOT_SMD:SOT-23-6
- added C23: 0.1uF, Capacitor_SMD:C_0402_1005Metric, F.Cu at (125.3, 94.9)
- added IC2: MIC23050-SYML-TR, SamacSys_Parts:SON50P200X200X90-9N-D, F.Cu at (122.7, 93.1)
- added R16: 1k, Resistor_SMD:R_0402_1005Metric, F.Cu at (115.2, 105.2)
- added R18: 1, Resistor_SMD:R_0402_1005Metric, F.Cu at (116.2, 102.3)
- added R19: 1, Resistor_SMD:R_0402_1005Metric, F.Cu at (120.5, 101.1)
- C1, C10, C2, C3, R3: moved to B.Cu
- C16: value 10uF -> 0.1uF
- C17: value 0.1uF -> 10uF
- C18, C22: value 0.1uF -> 22nF
- C20: value 22nF -> 0.1uF
- C21: value 22nF -> 10uF
- C6: value 560pF -> 0.1uF
- C7: value 4.7uF -> 560pF
- C8: value 0.1uF -> 4.7uF; moved to B.Cu
- C9: value 4.7uF -> 0.1uF
- D2: moved to F.Cu
- IC1: value MIC23050-SYML-TR -> MMC5633NJL; footprint SamacSys_Parts:SON50P200X200X90-9N-D -> SamacSys_Parts:BGA4C40P2X2_85X85X60; moved to F.Cu
- J2: footprint Connector_JST:JST_PH_B2B-PH-K_1x02_P2.00mm_Vertical -> Connector_JST:JST_PH_S2B-PH-K_1x02_P2.00mm_Horizontal
- R1: value 10k -> 5.1k; moved to B.Cu
- R10, R11: value 5.1k -> 390k
- R12: value 1 -> 10k
- R13: value 1 -> 1k; moved to B.Cu
- R14, R15: value 1 -> 5.1k
- R2: value 261 -> 5.1k; moved to B.Cu
- R20: value 47k -> 1k
- R22, R23: value 1k -> 1
- R24: value 390k -> 47k
- R25: value 15k -> 47k
- R4: value 10k -> 261
- R6: value 390k -> 10k
- R8: value 10k -> 15k; moved to F.Cu
- R9: value 1k -> 10k; moved to F.Cu
- S1: value SSU-121BRT -> PCM12SMTR; footprint SamacSys_Parts:SSU121BRT -> SamacSys_Parts:PCM12SMTR
- moved C18 66.1 mm to (115.7, 106.6)
- moved J1 63.5 mm to (120.7, 109.7), turned to 0 degrees
- moved R24 60.2 mm to (116.2, 105.2), turned to -90 degrees
- moved C15 59.3 mm to (117.5, 106.6), turned to 180 degrees
- moved R1 57.4 mm to (125.5, 109.4)
- moved R2 53.9 mm to (125.3, 107.7)
- moved C8 53.4 mm to (123.9, 90.4), turned to -90 degrees
- moved R22 52.2 mm to (127.7, 105.3), turned to -90 degrees
- moved R20 51.0 mm to (128.6, 102.5), turned to 90 degrees
- moved C22 51.0 mm to (128.2, 101.1), turned to 180 degrees
- moved C16 49.6 mm to (119.4, 106.6), turned to 0 degrees
- moved R5 49.3 mm to (130.7, 105.6), turned to 180 degrees
- moved R25 49.0 mm to (127.7, 102.5), turned to 90 degrees
- moved L1 47.4 mm to (123.0, 90.5)
- moved C10 45.4 mm to (123.5, 87.2), turned to 90 degrees
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Connections:
- C10 pad 1: GND -> +BATT
- C10 pad 2: +BATT -> GND
- C15 pad 1: /MotorDriver1/EN -> /M_EN
- C16 pad 1: VDC -> /M_RST
- C17 pad 1: /MotorDriver0/EN -> VDC
- C18 pad 1: /MotorDriver1/RST -> Net-(C18-Pad1)
- C19 pad 1: /MotorDriver0/RST -> /M_EN
- C20 pad 1: Net-(C20-Pad1) -> /M_RST
- C21 pad 1: Net-(C21-Pad1) -> VDC
- C22 pad 1: /VREF -> Net-(C22-Pad1)
- C4 pad 1: /GPIO9 -> /VREF
- C5 pad 1: /VSENSE -> /GPIO9
- C6 pad 1: +3V3 -> /VSENSE
- C6 pad 2: /CFF -> GND
- C7 pad 1: VDC -> +3V3
- C7 pad 2: GND -> /CFF
- C8 pad 1: +5V -> VDC
- C9 pad 1: +BATT -> +5V
- L1 pad 2: Net-(IC1-SW) -> Net-(IC2-SW)
- R1 pad 2: /RST -> /SCL
- R10 pad 1: /CC1 -> VDC
- R10 pad 2: GND -> /VSENSE
- R11 pad 1: /CC2 -> /VSENSE
- R12 pad 1: Net-(U4-SENSEB) -> Net-(U3-PROG)
- R13 pad 1: Net-(U4-SENSEA) -> Net-(D2-K)
- R13 pad 2: GND -> Net-(U3-STAT)
- R14 pad 1: Net-(U5-SENSEB) -> /CC1
- R15 pad 1: Net-(U5-SENSEA) -> /CC2
- R2 pad 2: Net-(D1-A) -> /SDA
- R20 pad 1: Net-(U4-TOFF) -> Net-(U5-TOFF)
- R20 pad 2: GND -> Net-(C22-Pad1)
- R22 pad 1: Net-(U4-TOFF) -> Net-(U5-SENSEB)
- R22 pad 2: Net-(C20-Pad1) -> GND
- R23 pad 1: Net-(U5-TOFF) -> Net-(U5-SENSEA)
- R23 pad 2: Net-(C21-Pad1) -> GND
- R24 pad 1: VDC -> Net-(U4-TOFF)
- R24 pad 2: /VREF -> GND
- R25 pad 1: /VREF -> Net-(U5-TOFF)
- R3 pad 2: /GPIO8 -> /RST
- R4 pad 2: /GPIO2 -> Net-(D1-A)
- R5 pad 2: /GPIO9 -> /GPIO8
- R6 pad 1: VDC -> +3V3
- R6 pad 2: /VSENSE -> /GPIO2
- R7 pad 1: /VSENSE -> VDC
- R7 pad 2: GND -> /VREF
- R8 pad 1: Net-(U3-PROG) -> /VREF
- R9 pad 1: Net-(D2-K) -> +3V3
- R9 pad 2: Net-(U3-STAT) -> /GPIO9
- U1 pad 16: unconnected-(U1-IO10-Pad16) -> /M0_STEP
- U1 pad 18: unconnected-(U1-IO4-Pad18) -> /M0_DIR
- U1 pad 19: unconnected-(U1-IO5-Pad19) -> /M1_STEP
- U1 pad 20: unconnected-(U1-IO6-Pad20) -> /M1_DIR
- U1 pad 21: unconnected-(U1-IO7-Pad21) -> /M_EN
- U1 pad 6: unconnected-(U1-IO3-Pad6) -> /M_RST
- U4 pad 1: /MotorDriver1/DIR -> /M0_DIR
- U4 pad 10: /M1_B1 -> /M0_B1
- U4 pad 13: /MotorDriver1/EN -> /M_EN
- U4 pad 14: /MotorDriver1/RST -> /M_RST
- U4 pad 2: /MotorDriver1/STEP -> /M0_STEP
- U4 pad 3: /M1_A1 -> /M0_A1
- U4 pad 5: /M1_A2 -> /M0_A2
- U4 pad 8: /M1_B2 -> /M0_B2
- U5 pad 1: /MotorDriver0/DIR -> /M1_DIR
- U5 pad 10: /M0_B1 -> /M1_B1
- U5 pad 13: /MotorDriver0/EN -> /M_EN
- U5 pad 14: /MotorDriver0/RST -> /M_RST
- U5 pad 2: /MotorDriver0/STEP -> /M1_STEP
- U5 pad 3: /M0_A1 -> /M1_A1
- U5 pad 5: /M0_A2 -> /M1_A2
- U5 pad 8: /M0_B2 -> /M1_B2
Routing:
- net VDC: track 0.11 -> 77.1 mm, vias 0 -> 7
- net +3V3: track 2.24 -> 67.8 mm, vias 0 -> 13
- net +5V: track 1.44 -> 34.2 mm, vias 1 -> 3
- net /M_RST: track 0.00 -> 30.6 mm, vias 0 -> 3
- net /VREF: track 2.53 -> 29.6 mm, vias 0 -> 2
- net /M_EN: track 0.00 -> 22.1 mm, vias 0 -> 2
- net GND: track 18.1 -> 39.0 mm, vias 9 -> 21
- net +BATT: track 10.7 -> 28.8 mm, vias 1 -> 2
- net /M0_B2: track 0.61 -> 18.0 mm, vias 1 -> 2
- net /M0_A2: track 0.66 -> 17.8 mm, vias 1 -> 2
- net /M1_B1: track 0.00 -> 12.4 mm, vias 0 -> 2
- net /GPIO9: track 0.00 -> 12.0 mm, vias 0 -> 1
- net /SCL: track 0.00 -> 11.4 mm, vias 0 -> 1
- net /M0_A1: track 1.15 -> 12.4 mm, vias 1 -> 2
- net /SDA: track 0.00 -> 10.5 mm, vias 0 -> 1
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- added copper zone on In1.Cu, net +3V3
- added copper zone on In2.Cu, net +3V3
- added copper zone on B.Cu, net GND
- added copper zone on F.Cu, net GND
Other:
- board size 27.9 x 28 mm -> 21.2 x 28 mm
- board text added: "MiniBOT"
- board text added: "V3"

Commit message: refining pcb and simulator code
Parts:
- moved C1 6.44 mm to (120.0, 91.0), turned to 90 degrees
- moved C2 5.10 mm to (121.0, 91.0), turned to -90 degrees
- moved C10 3.79 mm to (122.9, 91.0), turned to -90 degrees
- moved C3 3.34 mm to (123.8, 91.0), turned to -90 degrees
- moved R3 2.32 mm to (124.8, 91.0), turned to -90 degrees
- moved C8 2.06 mm to (121.9, 91.0)
- moved R13 1.28 mm to (124.0, 89.6)
- moved U3 0.12 mm to (122.5, 87.4)
- moved R2 0.11 mm to (125.5, 107.7)
- moved D2 0.09 mm to (124.8, 88.4)
- moved L1 0.08 mm to (123.0, 90.6)
Routing:
- net +3V3: track 67.8 -> 63.3 mm, vias 13 -> 12
- net Net-(U3-STAT): track 8.14 -> 4.26 mm, vias 2 -> 1
- net VDC: track 77.1 -> 79.6 mm
- net GND: track 39.0 -> 40.9 mm
- net /RST: track 8.06 -> 9.75 mm
- net +BATT: track 28.8 -> 30.2 mm
Other:
- board text added: "- +"
- board text added: "3v3"
- board text added: "BOOT"
- board text added: "CHG"
- board text added: "RST"

Commit message: getting close to order state
Parts:
- removed R4: 261, Resistor_SMD:R_0402_1005Metric
- added J4: Conn_01x01, TestPoint:TestPoint_Pad_D1.0mm, B.Cu at (127.9, 90.8)
- added JP1: Jumper_3_Bridged12, Jumper:SolderJumper-3_P1.3mm_Bridged12_RoundedPad1.0x1.5mm, B.Cu at (117.5, 110.6)
- added JP2: Jumper_3_Bridged12, Jumper:SolderJumper-3_P1.3mm_Bridged12_RoundedPad1.0x1.5mm, B.Cu at (122.1, 111.1)
- added R17: 1k, Resistor_SMD:R_0402_1005Metric, F.Cu at (130.6, 92.8)
- moved C4 0.97 mm to (116.0, 97.2)
- moved R8 0.91 mm to (116.0, 98.2)
- moved U3 0.19 mm to (122.7, 87.5)
- moved L1 0.17 mm to (122.8, 90.6)
- moved R13 0.12 mm to (124.2, 89.6)
- moved D2 0.10 mm to (124.9, 88.4)
- turned R9 to -90 degrees
Connections:
- R7 pad 1: VDC -> +3V3
- U1 pad 12: unconnected-(U1-IO0-Pad12) -> /GPIO0
- U4 pad 15: +3V3 -> /MODE2
- U4 pad 16: GND -> /MODE1
- U5 pad 15: +3V3 -> /MODE2
- U5 pad 16: GND -> /MODE1
Routing:
- net +3V3: track 63.3 -> 43.7 mm, vias 12 -> 10
- net /MODE2: track 0.00 -> 19.0 mm, vias 0 -> 3
- net /MODE1: track 0.00 -> 14.5 mm, vias 0 -> 3
- net GND: track 40.9 -> 48.6 mm, vias 21 -> 22
- net /GPIO0: track 0.00 -> 5.02 mm
- net /M0_B2: track 18.0 -> 13.5 mm
- net VDC: track 79.6 -> 76.4 mm, vias 7 -> 5
- net /M_RST: track 30.6 -> 29.1 mm
- net /GPIO8: track 6.48 -> 7.91 mm
- net /VSENSE: track 5.33 -> 4.07 mm
- net /M_EN: track 22.1 -> 20.9 mm
- net /VREF: track 29.6 -> 28.8 mm
- net /SDA: track 10.6 -> 11.3 mm
- net /M0_A2: track 17.8 -> 18.4 mm
- net /M1_A2: track 8.29 -> 8.93 mm
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Other:
- board text added: "M1"
- board text added: "M2"
- board text removed: "MiniBOT"
- board text removed: "V3"
