File: pcb/MiniBot.kicad_sch (KiCad schematic)
At the start: 42 parts, among them IC1 MMC5633NJL, IC2 MIC23050-SYML-TR, J1 Conn_01x08, J2 Conn_01x02, J3 GSB1C41110SSHR, J4 Conn_01x01, U1 ESP32-C3-MINI-1-H4X, U3 MCP73832-2-OT

Commit message: testing coils, improved hall sensor integration, tons of cleanup
Parts:
- R8: value 15k -> 12.4k
Changed lines of the file:
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@@
       (effects (font (size 1.27 1.27)) (justify left))
     )
-    (property "Value" "15k" (at 158.75 114.3 0)
+    (property "Value" "12.4k" (at 158.75 114.3 0)
       (effects (font (size 1.27 1.27)) (justify left))
     )
