File: archived/pcb v3/MiniBot.kicad_pcb (KiCad board)
At the start: 4 copper layers, 21.2 x 28 mm, 60 parts, among them IC1 MMC5633NJL, IC2 MIC23050-SYML-TR, J1 Conn_01x08, J2 Conn_01x02, J3 GSB1C41110SSHR, J4 Conn_01x01, U1 ESP32-C3-MINI-1-H4X, U3 MCP73832-2-OT, U4 STSPIN220, U5 STSPIN220

Commit message: checkpoint before i break everything
Parts:
- J1: footprint Connector_Molex:Molex_PicoBlade_53047-0810_1x08_P1.25mm_Vertical -> Connector_JST:JST_SH_BM08B-SRSS-TB_1x08-1MP_P1.00mm_Vertical
- R17: value 5.1k -> 1k
- moved JP1 24.8 mm to (121.5, 111.2), turned to 180 degrees
- moved R1 6.77 mm to (119.0, 108.7), turned to 0 degrees
- moved JP2 5.38 mm to (116.3, 109.4), turned to -90 degrees
- moved J1 4.91 mm to (120.7, 109.7)
- moved R2 0.05 mm to (120.8, 107.7)
Connections:
- J1 pad 7: /M0_B2 -> /M0_B1
- J1 pad 8: /M0_B1 -> /M0_B2
Routing:
- net /MODE2: track 29.2 -> 36.5 mm
- net /MODE1: track 41.9 -> 35.9 mm
- net /M0_B1: track 13.0 -> 16.7 mm, vias 1 -> 2
- net GND: track 94.3 -> 96.6 mm, vias 24 -> 25
- net /M0_A1: track 7.89 -> 10.2 mm
- net /M0_A2: track 6.16 -> 8.33 mm
- net /M0_B2: track 10.7 -> 12.7 mm, vias 1 -> 2
- net /M1_A2: track 7.58 -> 8.85 mm
- net VDC: track 48.1 -> 49.3 mm
- net /M1_B2: track 7.17 -> 8.31 mm
- net +3V3: track 37.1 -> 38.2 mm, vias 12 -> 13
- net /M1_A1: track 8.72 -> 9.72 mm
- net /SCL: track 12.7 -> 13.6 mm
- net /M1_B1: track 14.6 -> 13.9 mm, vias 0 -> 2
