File: archived/pcb v3/MiniBot.kicad_sch (KiCad schematic)
At the start: 42 parts, among them IC1 MMC5633NJL, IC2 MIC23050-SYML-TR, J1 Conn_01x08, J2 Conn_01x02, J3 GSB1C41110SSHR, J4 Conn_01x01, U1 ESP32-C3-MINI-1-H4X, U3 MCP73832-2-OT

Commit message: checkpoint before i break everything
Parts:
- J1: footprint Connector_Molex:Molex_PicoBlade_53047-0810_1x08_P1.25mm_Vertical -> Connector_JST:JST_SH_BM08B-SRSS-TB_1x08-1MP_P1.00mm_Vertical
- R17: value 5.1k -> 1k
Connections:
- net M0_B1: now also J1.7 (Pin_7); no longer J1.8 (Pin_8)
- net M0_B2: now also J1.8 (Pin_8); no longer J1.7 (Pin_7)
Changed lines of the file:
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@@
+    (stroke (width 0) (type default))
+  )
+  (wire (pts (xy 143.51 29.21) (xy 146.05 29.21))
     (stroke (width 0) (type default))
   )
@@
     (stroke (width 0) (type default))
   )
+  (wire (pts (xy 143.51 31.75) (xy 144.78 31.75))
+    (stroke (width 0) (type default))
+  )
   (wire (pts (xy 186.69 115.57) (xy 186.69 116.84))
     (stroke (width 0) (type default))
@@
     (stroke (width 0) (type default))
   )
+  (wire (pts (xy 144.78 55.88) (xy 144.78 31.75))
+    (stroke (width 0) (type default))
+  )
   (wire (pts (xy 115.57 21.59) (xy 116.84 21.59))
     (stroke (width 0) (type default))
@@
     (stroke (width 0) (type default))
   )
-  (wire (pts (xy 143.51 31.75) (xy 144.78 31.75))
-    (stroke (width 0) (type default))
-  )
   (wire (pts (xy 31.75 40.64) (xy 27.94 40.64))
     (stroke (width 0) (type default))
@@
     (stroke (width 0) (type default))
   )
-  (wire (pts (xy 146.05 29.21) (xy 146.05 55.88))
+  (wire (pts (xy 146.05 29.21) (xy 146.05 53.34))
     (stroke (width 0) (type default))
   )
@@
     (stroke (width 0) (type default))
   )
+  (wire (pts (xy 160.02 55.88) (xy 144.78 55.88))
+    (stroke (width 0) (type default))
+  )
   (wire (pts (xy 91.44 63.5) (xy 91.44 66.04))
     (stroke (width 0) (type default))
@@
     (stroke (width 0) (type default))
   )
-  (wire (pts (xy 144.78 53.34) (xy 160.02 53.34))
-    (stroke (width 0) (type default))
-  )
   (wire (pts (xy 54.61 134.62) (xy 54.61 137.16))
     (stroke (width 0) (type default))
@@
     (stroke (width 0) (type default))
   )
-  (wire (pts (xy 143.51 29.21) (xy 146.05 29.21))
-    (stroke (width 0) (type default))
-  )
   (wire (pts (xy 31.75 29.21) (xy 27.94 29.21))
     (stroke (width 0) (type default))
@@
     (stroke (width 0) (type default))
   )
-  (wire (pts (xy 146.05 55.88) (xy 160.02 55.88))
-    (stroke (width 0) (type default))
-  )
   (wire (pts (xy 140.97 162.56) (xy 140.97 171.45))
     (stroke (width 0) (type default))
@@
     (stroke (width 0) (type default))
   )
-  (wire (pts (xy 144.78 31.75) (xy 144.78 53.34))
-    (stroke (width 0) (type default))
-  )
   (wire (pts (xy 143.51 64.77) (xy 149.86 64.77))
     (stroke (width 0) (type default))
@@
   )
   (wire (pts (xy 55.88 35.56) (xy 54.61 35.56))
+    (stroke (width 0) (type default))
+  )
+  (wire (pts (xy 146.05 53.34) (xy 160.02 53.34))
     (stroke (width 0) (type default))
   )
@@
     (effects (font (size 1.27 1.27)) (justify right bottom))
   )
-  (label "M0_B1" (at 157.48 55.88 180) (fields_autoplaced)
+  (label "M0_B1" (at 157.48 53.34 180) (fields_autoplaced)
     (effects (font (size 1.27 1.27)) (justify right bottom))
   )
@@
     (effects (font (size 1.27 1.27)) (justify right bottom))
   )
-  (label "M0_B2" (at 157.48 53.34 180) (fields_autoplaced)
+  (label "M0_B2" (at 157.48 55.88 180) (fields_autoplaced)
     (effects (font (size 1.27 1.27)) (justify right bottom))
   )
@@
       (effects (font (size 1.27 1.27)))
     )
-    (property "Value" "5.1k" (at 140.97 100.33 90)
+    (property "Value" "1k" (at 140.97 100.33 90)
       (effects (font (size 1.27 1.27)))
     )
@@
       (effects (font (size 1.27 1.27)) (justify left))
     )
-    (property "Footprint" "Connector_Molex:Molex_PicoBlade_53047-0810_1x08_P1.25mm_Vertical" (at 165.1 45.72 0)
-      (effects (font (size 1.27 1.27)) hide)
-    )
+    (property "Footprint" "Connector_JST:JST_SH_BM08B-SRSS-TB_1x08-1MP_P1.00mm_Vertical" (at 165.1 45.72 0)
+      (effects (font (size 1.27 1.27)) hide)
+    )
