File: pcbs/MiniBot_MainBoard/MiniBot.kicad_sch (KiCad schematic)
At the start: 42 parts, among them IC1 MMC5633NJL, IC2 MIC23050-SYML-TR, J1 Conn_01x08, J2 Conn_01x02, J3 GSB1C41110SSHR, J4 Conn_01x01, U1 ESP32-C3-MINI-1-H4X, U3 MCP73832-2-OT

Commit message: led updates
Parts:
- removed D1, D2: LED, Diode_SMD:D_0402_1005Metric, symbol Device:LED
- removed J4: Conn_01x01, TestPoint:TestPoint_Pad_D1.0mm, symbol Connector_Generic:Conn_01x01
- removed R17: 5.1k, Resistor_SMD:R_0402_1005Metric, symbol Device:R
- added LED1: EASV2010RWA0, EASV2010RWA0, symbol SamacSys_Parts:EASV2010RWA0
- added R4: 10k, Resistor_SMD:R_0402_1005Metric, symbol Device:R
Connections:
- net +BATT: now also LED1.3 (R6+)
- net GND: now also R4.2
- net LED_R: now reaches R13.1
- net LED_R: now also LED1.4 (R6-)
- net GPIO0 renamed LED_W
- net LED_W: now also LED1.1 (T1+)
- new net: LED1.2 (T1-), R4.1
Other:
- moved on the sheet: C10, C3, C4, C5, C6, J1, J2, JP1, JP2, R1, R10, R11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

Commit message: cleanup minibot schematic
Other:
- note added: "Battery"
- note added: "ESP32-C3"
- note added: "LEDs"
- note added: "Mag Sensor"
- note added: "Power & Regulation"
- note added: "Steppers"
- note added: "USB"
- moved on the sheet: C1, C2, C3, C4, C5, C6, IC1, J1, J2, JP1, JP2, LED1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

Commit message: mostly finished server pcb, added pogo charge pins to bots, started charge case pcb
Parts:
- added TP1, TP2: TestPoint, TestPoint:TestPoint_Pad_D1.0mm, symbol Connector:TestPoint
Connections:
- net +5V: now also TP2.1
- net GND: now also TP1.1
Changed lines of the file:
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@@
+    (stroke (width 0) (type default))
+  )
+  (wire (pts (xy 167.64 50.8) (xy 167.64 53.34))
     (stroke (width 0) (type default))
   )
@@
   )
   (wire (pts (xy 127 170.18) (xy 123.19 170.18))
+    (stroke (width 0) (type default))
+  )
+  (wire (pts (xy 175.26 50.8) (xy 175.26 53.34))
     (stroke (width 0) (type default))
   )
@@
     )
   )
+  (symbol (lib_id "Connector:TestPoint") (at 167.64 50.8 0) (unit 1)
+    (in_bom yes) (on_board yes) (dnp no)
+    (property "Reference" "TP2" (at 166.37 44.45 0)
+      (effects (font (size 1.27 1.27)) (justify left))
+    )
+    (property "Value" "TestPoint" (at 163.83 41.91 0)
+      (effects (font (size 1.27 1.27)) (justify left))
+    )
+    (property "Footprint" "TestPoint:TestPoint_Pad_D1.0mm" (at 172.72 50.8 0)
+      (effects (font (size 1.27 1.27)) hide)
+    )
+    (property "Datasheet" "~" (at 172.72 50.8 0)
+      (effects (font (size 1.27 1.27)) hide)
+    )
+    (pin "1")
+    (instances
+      (project "MiniBot"
+        (path "/0e598331-3211-4e8a-a305-31a83585854d"
+          (reference "TP2") (unit 1)
+        )
+      )
+    )
+  )
+  (symbol (lib_id "Connector:TestPoint") (at 175.26 50.8 0) (unit 1)
+    (in_bom yes) (on_board yes) (dnp no)
+    (property "Reference" "TP1" (at 177.8 44.45 0)
+      (effects (font (size 1.27 1.27)) (justify left))
+    )
+    (property "Value" "TestPoint" (at 175.26 41.91 0)
+      (effects (font (size 1.27 1.27)) (justify left))
+    )
+    (property "Footprint" "TestPoint:TestPoint_Pad_D1.0mm" (at 180.34 50.8 0)
+      (effects (font (size 1.27 1.27)) hide)
+    )
+    (property "Datasheet" "~" (at 180.34 50.8 0)
+      (effects (font (size 1.27 1.27)) hide)
+    )
+    (pin "1")
+    (instances
+      (project "MiniBot"
+        (path "/0e598331-3211-4e8a-a305-31a83585854d"
+          (reference "TP1") (unit 1)
+        )
+      )
+    )
+  )
   (symbol (lib_id "power:GND") (at 34.29 27.94 0) (unit 1)
     (in_bom yes) (on_board yes) (dnp no)
@@
     )
   )
+  (symbol (lib_id "power:GND") (at 175.26 53.34 0) (unit 1)
+    (in_bom yes) (on_board yes) (dnp no) (fields_autoplaced)
+    (property "Reference" "#PWR045" (at 175.26 59.69 0)
+      (effects (font (size 1.27 1.27)) hide)
+    )
+    (property "Value" "GND" (at 175.26 58.42 0)
+      (effects (font (size 1.27 1.27)))
+    )
+    (property "Footprint" "" (at 175.26 53.34 0)
+      (effects (font (size 1.27 1.27)) hide)
+    )
+    (property "Datasheet" "" (at 175.26 53.34 0)
+      (effects (font (size 1.27 1.27)) hide)
+    )
+    (pin "1")
+    (instances
+      (project "MiniBot"
+        (path "/0e598331-3211-4e8a-a305-31a83585854d"
+          (reference "#PWR045") (unit 1)
+        )
+      )
+    )
+  )
   (symbol (lib_id "power:GND") (at 194.31 29.21 0) (unit 1)
     (in_bom yes) (on_board yes) (dnp no) (fields_autoplaced)
@@
         )
       )
+    )
+  )
+  (symbol (lib_id "power:+5V") (at 167.64 53.34 180) (unit 1)
+    (in_bom yes) (on_board yes) (dnp no)
+    (property "Reference" "#PWR017" (at 167.64 49.53 0)
+      (effects (font (size 1.27 1.27)) hide)
+    )
+    (property "Value" "+5V" (at 167.64 58.42 0)
+      (effects (font (size 1.27 1.27)))
+    )
+    (property "Footprint" "" (at 167.64 53.34 0)
+      (effects (font (size 1.27 1.27)) hide)
+    )
+    (property "Datasheet" "" (at 167.64 53.34 0)
+      (effects (font (size 1.27 1.27)) hide)
+    )
+    (pin "1")
+    (instances
+      (project "MiniBot"
+        (path "/0e598331-3211-4e8a-a305-31a83585854d"
+          (reference "#PWR017") (unit 1)
+        )
+      )
